File: Historia-debugger.kicad_pcb (KiCad board)
At the start: 2 copper layers, 80 x 50 mm, 47 parts, among them J1 Conn_01x04_Female, J2 USB_B_Mini, SW1 SW_Push, SW2 SW_Push, SW3 SW_Push, SW4 SW_Push, SW6 SW_SPDT, U1 MCP2221-I_SL, U2 ATmega328-AU-MCU_Microchip_AT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, U3 Adafruit_938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

Commit message: rename PCB name
Parts:
- renumbered C3 to 0.1u, C4 to 47u
Changed lines of the file:
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@@
-(kicad_pcb (version 20171130) (host pcbnew "(5.1.8)-1")
+(kicad_pcb (version 20171130) (host pcbnew "(5.1.8-0-10_14)")
   (general
     (thickness 1.6)
@@
   (page A4)
   (layers
-    (0 F.Cu signal)
-    (31 B.Cu signal)
+    (0 F.Cu signal hide)
+    (31 B.Cu signal hide)
     (32 B.Adhes user)
     (33 F.Adhes user)
@@
     (tags "capacitor electrolytic")
     (attr smd)
-    (fp_text reference C4 (at 0 -4.35) (layer F.SilkS)
+    (fp_text reference 47u (at 0 4.318) (layer F.SilkS)
       (effects (font (size 1 1) (thickness 0.15)))
     )
@@
     (tags capacitor)
     (attr smd)
-    (fp_text reference C3 (at 0 -1.43) (layer F.SilkS)
+    (fp_text reference 0.1u (at 0 -1.43) (layer F.SilkS)
       (effects (font (size 1 1) (thickness 0.15)))
     )

Commit message: add silks and QR
Other:
- board text added: "Historia-Debugger"
- board text added: "[DESCRIPTION] This board is a debugger for Historia Motor Driver."
- board text removed: "Alice-F3000-Debugger"
- board text removed: "[DESCRIPTION] This board is a debugger for Alice-F3000 Motor Driver."
